File: Infineon.EVAL-2HS01G-300W-1.kicad_pcb (KiCad board)
At the start: 2 copper layers, 0 parts

Commit message: Update PCB design files
* Replace Top Copper picture which was in gray levels with its colored
  version.
* Add Edge Cuts so PCB 3D visualization is of accurate dimensions.
* Add some Throug Holes components land patttern to the User Comments
  layer in order to ease components placement later on.
Other:
- board outline added: 140 x 85 mm
- board text added: "+12V"
- board text added: "SGND"
